Commit message: feat: robot draw implementation

File: resources/simple.urdf (robot description, URDF)
Before this commit: robot robot, 4 links, 3 joints
Links:
- link humerus: geometry visual box size=0.25 0.25 2.5

Commit message: feat: draw collisions as wireframes

File: resources/simple.urdf (robot description, URDF)
Before this commit: robot robot, 4 links, 3 joints
Links:
- link ulna: geometry collision box size=2 2 2; visual cylinder length=0.6 radius=0.3
