Commit message: feat: implement mesh geometry loading with package:// path resolution
Parse <mesh filename="..."/> from URDF XML, resolve package:// paths by
walking up to find package.xml, and serialize mesh elements back on export.
Rename LoadModelFromCollada to LoadModelFromFile, fix assimp mesh import
(normals, index types, materials, GPU upload, node transforms). Update
R2D2 URDF to use actual gripper DAE meshes from the ROS urdf_tutorial.

File: resources/r2d2.urdf (robot description, URDF)
Before this commit: robot visual, 16 links, 15 joints
Links:
- link left_gripper: geometry visual mesh filename=package://urdf_tutorial/meshes/l_finger.dae
- link left_tip: geometry visual mesh filename=package://urdf_tutorial/meshes/l_finger_tip.dae
- link right_gripper: geometry visual mesh filename=package://urdf_tutorial/meshes/l_finger.dae
- link right_tip: geometry visual mesh filename=package://urdf_tutorial/meshes/l_finger_tip.dae
